File: a2-display/a2-display.brd (EAGLE design)
At the start: 160 x 97.5 mm, 52 parts, among them IC1 HT1632C

Commit message: stuff
Parts:
- moved IC1 25.4 mm to (84.5, 82.5)
- moved R13 9.23 mm to (92.5, 66.0), turned to 180 degrees
- moved R16 9.11 mm to (92.6, 43.2), turned to 180 degrees
- moved R15 8.98 mm to (92.7, 50.8), turned to 180 degrees
- moved R14 8.98 mm to (92.7, 58.4), turned to 180 degrees
- moved R11 7.73 mm to (77.5, 50.8), turned to 0 degrees
- moved R10 7.73 mm to (77.5, 58.4), turned to 0 degrees
- moved R9 7.47 mm to (77.2, 66.0), turned to 0 degrees
- moved R12 7.47 mm to (77.2, 43.2), turned to 0 degrees
- moved R20 6.85 mm to (109.9, 43.2), turned to 0 degrees
- moved R19 6.75 mm to (110.0, 50.7), turned to 0 degrees
- moved R18 6.33 mm to (110.4, 58.4), turned to 0 degrees
- moved R17 6.16 mm to (110.2, 66.0), turned to 0 degrees
- moved R4 5.37 mm to (44.8, 43.2), turned to 0 degrees
- moved R8 5.25 mm to (60.5, 43.2), turned to 180 degrees
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Routing:
- net R7R: track 149.1 -> 89.5 mm, vias 4 -> 2
- net R3R: track 122.9 -> 85.2 mm
- net R6G: track 146.6 -> 109.4 mm, vias 3 -> 2
- net R2G: track 132.6 -> 97.5 mm, vias 1 -> 2
- net N$10: track 7.61 -> 40.5 mm, vias 0 -> 2
- net N$11: track 18.3 -> 49.1 mm, vias 0 -> 2
- net R3G: track 121.6 -> 91.3 mm
- net R5R: track 79.1 -> 106.5 mm
- net R6R: track 69.9 -> 96.1 mm
- net R5G: track 89.6 -> 114.4 mm, vias 3 -> 2
- net N$12: track 34.3 -> 58.0 mm, vias 0 -> 2
- net R4R: track 97.2 -> 77.6 mm, vias 1 -> 2
- net R1G: track 84.5 -> 103.6 mm, vias 0 -> 3
- net R8G: track 75.8 -> 94.8 mm
- net N$1: track 59.1 -> 41.2 mm
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Other:
- outline, holes or cut-outs redrawn
